Commit message: rvis integration

File: robokoko/urdf/robokoko.xacro (robot description, xacro)
@@ -14,4 +14,10 @@
   	<material>Gazebo/Gray</material>
 	</gazebo>
+	<material name="yellow">
+		<color rgba="1 1 0 1"/>
+  </material>
+	<material name="black">
+   	<color rgba="0 0 0 1"/>
+  </material>
   <link name="robot_footprint"></link>
 	<!-- Chassis  -->
@@ -27,7 +33,7 @@
       <origin xyz="0.0 0 0" rpy=" 0 0 0"/>
       <inertia
-          ixx="0.1" ixy="0" ixz="0"
-          iyy="0.1" iyz="0"
-          izz="0.1"
+          ixx="0.00043333333333333337" ixy="0" ixz="0"
+          iyy="0.002033333333333333" iyz="0"
+          izz="0.0024333333333333334"
       />
     </inertial>
@@ -43,7 +49,5 @@
         <box size="0.22 .10 .02"/>
       </geometry>
-			<material name="blue">
-      	<color rgba="0 0 .8 1"/>
-      </material>
+			<material name="black"/>
 		</visual>
   </link>
@@ -62,7 +66,7 @@
 			<origin xyz="0.0 0 0" rpy="0 1.5707 1.5707"/>
 			<inertia
-			  ixx="0.0135" ixy="0" ixz="0"
-			  iyy="0.0135" iyz="0"
-			  izz="0.025"
+			  ixx="0.000135" ixy="0" ixz="0"
+			  iyy="0.000135" iyz="0"
+			  izz="9e-05"
 			/>
 		</inertial>
@@ -77,6 +81,6 @@
 			<geometry>
 				<cylinder radius="0.03" length="0.03"/>
-			</geometry>
-			<material name="yellow"/>
+				</geometry>
+				<material name="yellow"/>
 		</visual>
 	</link>
@@ -95,7 +99,7 @@
 			<origin xyz="0.0 0 0" rpy="0 1.5707 1.5707"/>
 			<inertia
-			  ixx="0.0135" ixy="0" ixz="0"
-			  iyy="0.0135" iyz="0"
-			  izz="0.025"
+			  ixx="0.000135" ixy="0" ixz="0"
+			  iyy="0.000135" iyz="0"
+			  izz="9e-05"
 			/>
 		</inertial>
@@ -128,7 +132,7 @@
 			<origin xyz="0.0 0 0" rpy="0 1.5707 1.5707"/>
 			<inertia
-			  ixx="0.0135" ixy="0" ixz="0"
-			  iyy="0.0135" iyz="0"
-			  izz="0.025"/>
+			  ixx="1.6e-05" ixy="0" ixz="0"
+			  iyy="1.6e-05" iyz="0"
+			  izz="1.6e-05"/>
 		</inertial>
 		<collision name='back_caster_collision'>

Commit message: Correct the robot inclination

File: robokoko/urdf/robokoko.xacro (robot description, xacro)
@@ -129,10 +129,10 @@
 	<link name='back_caster'>
 		<inertial>
-			<mass value="0.1"/>
+			<mass value="0.3"/>
 			<origin xyz="0.0 0 0" rpy="0 1.5707 1.5707"/>
 			<inertia
-			  ixx="1.6e-05" ixy="0" ixz="0"
-			  iyy="1.6e-05" iyz="0"
-			  izz="1.6e-05"/>
+			  ixx="4.8e-05" ixy="0" ixz="0"
+			  iyy="4.8e-05" iyz="0"
+			  izz="4.8e-05"/>
 		</inertial>
 		<collision name='back_caster_collision'>

Commit message: Add camera to robot

File: robokoko/urdf/robokoko.xacro (robot description, xacro)
@@ -3,4 +3,7 @@
 	<xacro:include filename="$(find robokoko)/urdf/robokoko.gazebo" />
 	<gazebo reference="chassis">
+  	<material>Gazebo/Black</material>
+	</gazebo>
+	<gazebo reference="camera">
   	<material>Gazebo/Black</material>
 	</gazebo>
@@ -179,3 +182,33 @@
 		</visual>
 	</link>
+	<!-- Camera -->
+	<joint name="camera_joint" type="fixed" >
+		<parent link="chassis"/>
+		<child link="camera"/>
+		<origin xyz="0.11 0 0" rpy="0 0 0"/>
+	</joint>
+	<link name='camera'>
+		<inertial>
+			<mass value="0.1"/>
+			<origin xyz="0.0 0 0" rpy="0 0 0"/>
+			<inertia
+			  ixx="1e-6" ixy="0" ixz="0"
+			  iyy="1e-6" iyz="0"
+			  izz="1e-6"
+			/>
+		</inertial>
+		<collision name='collision'>
+			<origin xyz="0.0 0 0" rpy="0 0 0"/>
+			<geometry>
+				<box size="0.02 0.1 0.02"/>
+			</geometry>
+		</collision>
+		<visual name='camera_visual'>
+			<origin xyz="0.0 0 0" rpy="0 0 0"/>
+			<geometry>
+				<box size="0.02 0.1 0.02"/>
+			</geometry>
+			<material name="black"/>
+		</visual>
+	</link>
 </robot>
